File: hardware/pcb/qc3_trigger/qc3_trigger.sch (KiCad schematic (older format))
At the start: 12 parts, among them J1 USB_B_Micro, J2 Vout, U1 AMS1117-5.0, U2 ATtiny85V-10SU

Commit message: правки в схеме
Parts:
- C1, C2: footprint (none) -> Capacitor_SMD:C_0805_2012Metric
- J1: footprint (none) -> Connector_USB:USB_Micro-B_Molex_47346-0001
- J2: footprint (none) -> Connector_PinHeader_2.54mm:PinHeader_1x02_P2.54mm_Vertical
- R1, R2, R3, R4, R5, R6: footprint (none) -> Resistor_SMD:R_0805_2012Metric
Changed lines of the file:
@@
 F 0 "R1" H 2270 1646 50  0000 L CNN
 F 1 "10k" H 2270 1555 50  0000 L CNN
-F 2 "" V 2130 1600 50  0001 C CNN
+F 2 "Resistor_SMD:R_0805_2012Metric" V 2130 1600 50  0001 C CNN
 F 3 "~" H 2200 1600 50  0001 C CNN
 	1    2200 1600
@@
 F 0 "R2" H 2270 2196 50  0000 L CNN
 F 1 "1k5" H 2270 2105 50  0000 L CNN
-F 2 "" V 2130 2150 50  0001 C CNN
+F 2 "Resistor_SMD:R_0805_2012Metric" V 2130 2150 50  0001 C CNN
 F 3 "~" H 2200 2150 50  0001 C CNN
 	1    2200 2150
@@
 F 0 "R3" V 2250 1900 50  0000 C CNN
 F 1 "470" V 2350 1900 50  0000 C CNN
-F 2 "" V 2380 1850 50  0001 C CNN
+F 2 "Resistor_SMD:R_0805_2012Metric" V 2380 1850 50  0001 C CNN
 F 3 "~" H 2450 1850 50  0001 C CNN
 	1    2450 1850
@@
 F 0 "C1" H 3550 1800 50  0000 L CNN
 F 1 "100n" H 3500 1700 50  0000 L CNN
-F 2 "" H 3450 1800 50  0001 C CNN
+F 2 "Capacitor_SMD:C_0805_2012Metric" H 3450 1800 50  0001 C CNN
 F 3 "~" H 3450 1800 50  0001 C CNN
 	1    3450 1800
@@
 F 0 "C2" H 4342 1846 50  0000 L CNN
 F 1 "100n" H 4300 1750 50  0000 L CNN
-F 2 "" H 4250 1800 50  0001 C CNN
+F 2 "Capacitor_SMD:C_0805_2012Metric" H 4250 1800 50  0001 C CNN
 F 3 "~" H 4250 1800 50  0001 C CNN
 	1    4250 1800
@@
 F 0 "J1" H 1557 2067 50  0000 C CNN
 F 1 "USB_B_Micro" H 1557 1976 50  0000 C CNN
-F 2 "" H 1650 1550 50  0001 C CNN
+F 2 "Connector_USB:USB_Micro-B_Molex_47346-0001" H 1650 1550 50  0001 C CNN
 F 3 "~" H 1650 1550 50  0001 C CNN
 	1    1500 1600
@@
 F 0 "J2" H 4930 1392 50  0000 L CNN
 F 1 "Vout" H 4930 1301 50  0000 L CNN
-F 2 "" H 4850 1400 50  0001 C CNN
+F 2 "Connector_PinHeader_2.54mm:PinHeader_1x02_P2.54mm_Vertical" H 4850 1400 50  0001 C CNN
 F 3 "~" H 4850 1400 50  0001 C CNN
 	1    4850 1400
@@
 F 0 "R4" H 2870 1646 50  0000 L CNN
 F 1 "10k" H 2870 1555 50  0000 L CNN
-F 2 "" V 2730 1600 50  0001 C CNN
+F 2 "Resistor_SMD:R_0805_2012Metric" V 2730 1600 50  0001 C CNN
 F 3 "~" H 2800 1600 50  0001 C CNN
 	1    2800 1600
@@
 F 0 "R5" H 2870 2196 50  0000 L CNN
 F 1 "1k5" H 2870 2105 50  0000 L CNN
-F 2 "" V 2730 2150 50  0001 C CNN
+F 2 "Resistor_SMD:R_0805_2012Metric" V 2730 2150 50  0001 C CNN
 F 3 "~" H 2800 2150 50  0001 C CNN
 	1    2800 2150
@@
 F 0 "R6" V 2850 1900 50  0000 C CNN
 F 1 "470" V 2950 1900 50  0000 C CNN
-F 2 "" V 2980 1850 50  0001 C CNN
+F 2 "Resistor_SMD:R_0805_2012Metric" V 2980 1850 50  0001 C CNN
 F 3 "~" H 3050 1850 50  0001 C CNN
 	1    3050 1850

Commit message: поменял местами dppin и dnpin
Parts:
- added J3: USB_A, Connector_USB:USB_A_CNCTech_1001-011-01101_Horizontal, symbol Connector:USB_A
Connections:
- wire segments 43 -> 53
- no-connect marks 6 -> 7
Changed lines of the file:
@@
 Connection ~ 2200 1400
 Wire Wire Line
-	1800 1600 2100 1600
+	1800 1600 1900 1600
 Wire Wire Line
 	2100 1600 2100 1850
@@
 Connection ~ 2800 1850
 Wire Wire Line
-	1800 1700 2050 1700
+	1800 1700 1950 1700
 Wire Wire Line
 	2050 1700 2050 1950
@@
 Connection ~ 1950 1400
 Wire Wire Line
-	1950 1400 1800 1400
+	1950 1400 1850 1400
 NoConn ~ 1800 1800
 NoConn ~ 1400 2000
@@
 NoConn ~ 3900 2750
 NoConn ~ 3900 3050
+$Comp
+L Connector:USB_A J3
+U 1 1 61438836
+P 1500 2750
+F 0 "J3" H 1557 3217 50  0000 C CNN
+F 1 "USB_A" H 1557 3126 50  0000 C CNN
+F 2 "Connector_USB:USB_A_CNCTech_1001-011-01101_Horizontal" H 1650 2700 50  0001 C CNN
+F 3 " ~" H 1650 2700 50  0001 C CNN
+	1    1500 2750
+	1    0    0    -1
+$EndComp
 Wire Wire Line
-	2650 1850 2650 2950
+	1800 2550 1850 2550
 Wire Wire Line
-	2650 2950 3900 2950
+	1850 2550 1850 1400
+Connection ~ 1850 1400
 Wire Wire Line
-	3250 1850 3250 2850
+	1850 1400 1800 1400
 Wire Wire Line
-	3250 2850 3900 2850
+	1800 2750 1900 2750
+Wire Wire Line
+	1900 2750 1900 1600
+Connection ~ 1900 1600
+Wire Wire Line
+	1900 1600 2100 1600
+Wire Wire Line
+	1800 2850 1950 2850
+Wire Wire Line
+	1950 2850 1950 1700
+Connection ~ 1950 1700
+Wire Wire Line
+	1950 1700 2050 1700
+$Comp
+L power:GND #PWR010
+U 1 1 6143CCDD
+P 1500 3200
+F 0 "#PWR010" H 1500 2950 50  0001 C CNN
+F 1 "GND" H 1505 3027 50  0000 C CNN
+F 2 "" H 1500 3200 50  0001 C CNN
+F 3 "" H 1500 3200 50  0001 C CNN
+	1    1500 3200
+	1    0    0    -1
+$EndComp
+Wire Wire Line
+	1500 3150 1500 3200
+NoConn ~ 1400 3150
+Wire Wire Line
+	2650 1850 2650 2850
+Wire Wire Line
+	2650 2850 3900 2850
+Wire Wire Line
+	3250 1850 3250 2950
+Wire Wire Line
+	3250 2950 3900 2950
 $EndSCHEMATC

Commit message: вариант с повернутой тинькой
Changed lines of the file:
@@
 NoConn ~ 1400 3150
 Wire Wire Line
-	2650 1850 2650 2850
+	2650 1850 2650 2950
 Wire Wire Line
-	2650 2850 3900 2850
+	2650 2950 3900 2950
 Wire Wire Line
-	3250 1850 3250 2950
+	3250 1850 3250 2850
 Wire Wire Line
-	3250 2950 3900 2950
+	3250 2850 3900 2850
 $EndSCHEMATC
